File: watch-board/watch-board.kicad_pcb (KiCad board)
At the start: 2 copper layers, 34 x 34 mm, 64 parts, among them J1 Conn_PAD, J2 Conn_PAD, J3 Conn_PAD, J4 Conn_PAD, J5 Conn_PAD, Q1 Phototransistor_ALS-PT19-315C, Q2 Phototransistor_ALS-PT19-315C, Q3 Transistor_MMBT3904-TP, U1 Display-Driver_PCA8561ANH, U2 Regulator_BQ25504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

Commit message: all wiring done except gnd
Parts:
- S1: moved to B.Cu
- moved S1 13.9 mm to (147.8, 108.8)
- moved R14 11.4 mm to (152.9, 108.0), turned to 90 degrees
- moved R21 9.93 mm to (144.0, 114.9), turned to 0 degrees
- moved R13 8.97 mm to (150.9, 108.0), turned to 90 degrees
- moved C19 6.54 mm to (143.0, 110.7), turned to 90 degrees
- moved R12 4.49 mm to (128.2, 94.8), turned to 90 degrees
- moved R19 4.03 mm to (145.0, 110.7), turned to 90 degrees
- moved C4 3.92 mm to (129.1, 89.9), turned to 180 degrees
- moved R11 3.42 mm to (126.2, 94.8), turned to 90 degrees
- moved C6 2.87 mm to (150.2, 90.4), turned to 90 degrees
- moved C10 2.52 mm to (135.5, 99.1)
- moved C11 2.52 mm to (135.5, 101.1)
- moved Q1 2.23 mm to (135.0, 111.0)
- moved Q2 2.16 mm to (145.0, 111.0), turned to 270 degrees
- moved C16 1.76 mm to (135.5, 96.4), turned to 90 degrees
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Connections:
- C3 pad 2: Net-(C3-Pad2) -> GND
- C4 pad 2: Net-(C4-Pad2) -> GND
- DS1 pad 2: /1G -> GND
- DS2 pad 2: /1G -> GND
- U1 pad 12: /1G -> GND
- U1 pad 2: Net-(C4-Pad2) -> VDD
- U1 pad 3: Net-(C3-Pad2) -> VDD
- U4 pad 11: /VLIGHT_L -> /LIGHT_L
- U4 pad 12: /VLIGHT_R -> /VLIGHT_L
- U4 pad 8: /LIGHT_L -> /LIGHT_R
- U4 pad 9: /LIGHT_R -> /VLIGHT_R
Routing:
- net VDD: track 0.00 -> 136.3 mm, vias 0 -> 3
- net GND: track 0.00 -> 91.8 mm, vias 0 -> 4
- net /LIGHT_R: track 0.00 -> 41.3 mm, vias 0 -> 2
- net /1G: track 39.2 -> 0.00 mm
- net /VBAT_OK: track 0.00 -> 33.8 mm, vias 0 -> 2
- net /VLIGHT_R: track 0.00 -> 32.8 mm, vias 0 -> 1
- net Net-(C2-Pad1): track 0.00 -> 30.7 mm, vias 0 -> 1
- net Net-(R1-Pad1): track 0.00 -> 30.4 mm, vias 0 -> 2
- net /BUTTON: track 0.00 -> 27.7 mm, vias 0 -> 2
- net /RESET: track 0.00 -> 27.0 mm, vias 0 -> 1
- net /SCL: track 0.00 -> 24.2 mm, vias 0 -> 1
- net /SDA: track 0.00 -> 18.5 mm, vias 0 -> 1
- net /LOAD: track 0.00 -> 18.5 mm
- net /LIGHT: track 0.00 -> 16.3 mm
- net /LIGHT_L: track 0.00 -> 14.2 mm
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- added copper zone on B.Cu, net Net-(C2-Pad1)
- added copper zone on B.Cu, net Net-(L1-Pad2)

Commit message: finished wiring
Parts:
- moved BZ1 0.54 mm to (141.0, 105.5)
- moved C19 0.35 mm to (143.0, 111.1)
- moved R21 0.34 mm to (144.0, 114.6)
- moved R22 0.29 mm to (140.0, 113.3)
- moved R15 0.26 mm to (140.0, 115.3)
- moved C12 0.10 mm to (125.8, 97.6)
- moved C13 0.10 mm to (125.8, 99.5)
Connections:
- DS1 pad 2: GND -> /1G
- DS2 pad 2: GND -> /1G
- U1 pad 12: GND -> /1G
- U1 pad 31: /COM2 -> Net-(U1-Pad31)
- U1 pad 32: /COM1 -> Net-(U1-Pad32)
Routing:
- net GND: track 91.8 -> 135.9 mm, vias 4 -> 13
- net /1G: track 0.00 -> 39.2 mm
- net /VBAT_OK: track 33.8 -> 51.5 mm, vias 2 -> 4
- net Net-(R1-Pad1): track 30.4 -> 15.8 mm
- net Net-(Q1-Pad2): track 2.80 -> 9.17 mm, vias 0 -> 1
- net Net-(L1-Pad2): track 0.00 -> 4.83 mm
- net Net-(D1-Pad2): track 8.44 -> 5.42 mm
- net VDD: track 136.3 -> 138.3 mm, vias 3 -> 5
- net /LIGHT_R: track 41.3 -> 43.1 mm
- net /RESET: track 27.0 -> 28.8 mm
- net Net-(C2-Pad1): track 30.7 -> 29.1 mm
- net /COM1: track 36.5 -> 35.3 mm
- net /SCL: track 24.2 -> 25.4 mm
- net /SDA: track 18.5 -> 19.6 mm
- net /VLIGHT_R: track 32.8 -> 33.3 mm
- added copper zone on F.Cu, net GND
