File: watch-board/watch-board.kicad_pcb (KiCad board)
At the start: 4 copper layers, 34 x 34 mm, 64 parts, among them J1 Conn_PAD, J2 Conn_PAD, J3 Conn_PAD, J4 Conn_PAD, J5 Conn_PAD, Q1 Phototransistor_ALS-PT19-315C, Q2 Phototransistor_ALS-PT19-315C, Q3 Transistor_MMBT3904-TP, U1 Display-Driver_PCA8561ANH, U2 Regulator_BQ25504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

Commit message: downloaded possible silk screen graphic
Other:
- board text added: "2020"
- board text added: "Luke Nonas-Hunter"

Commit message: added silk screen
Parts:
- added G***: LOGO, luke-footprints:Silk-Screen_Clock, F.Cu at (147.1, 93.8)

Commit message: connecting chain to ground
Routing:
- net GND: track 128.9 -> 130.7 mm, vias 16 -> 17
Changed lines of the file:
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@@
     (thickness 1.6)
     (drawings 9)
-    (tracks 785)
+    (tracks 788)
     (zones 0)
     (modules 65)
@@
     (1 In1.Cu power hide)
     (2 In2.Cu power hide)
-    (31 B.Cu signal hide)
+    (31 B.Cu signal)
     (32 B.Adhes user hide)
     (33 F.Adhes user hide)
@@
   )
   (setup
-    (last_trace_width 0.2)
+    (last_trace_width 0.5)
     (user_trace_width 0.2)
     (user_trace_width 0.3)
@@
   (segment (start 141.1479 92.0303) (end 141.8979 91.2803) (width 0.2) (layer B.Cu) (net 2))
   (segment (start 140.4104 92.0303) (end 141.1479 92.0303) (width 0.2) (layer B.Cu) (net 2))
-  (segment (start 142.8279 90.5503) (end 142.0779 91.3003) (width 0.2) (layer B.Cu) (net 2))
   (segment (start 143.5654 90.5503) (end 142.8279 90.5503) (width 0.2) (layer B.Cu) (net 2))
   (segment (start 142.8279 92.0503) (end 142.0779 91.3003) (width 0.2) (layer B.Cu) (net 2))
@@
   (segment (start 132.61506 110.51506) (end 132.61506 110.01248) (width 0.2) (layer B.Cu) (net 2))
   (segment (start 133.4 111.3) (end 132.61506 110.51506) (width 0.2) (layer B.Cu) (net 2))
+  (segment (start 142.8279 90.5503) (end 142.0779 91.3003) (width 0.2) (layer B.Cu) (net 2))
+  (segment (start 142.21186 85.49564) (end 143.5 84.2075) (width 0.5) (layer B.Cu) (net 2))
+  (segment (start 143.5 84.2075) (end 143.5 84.2075) (width 0.5) (layer B.Cu) (net 2))
+  (via (at 143.5 84.2075) (size 0.8) (drill 0.4) (layers F.Cu B.Cu) (net 2))
   (segment (start 131.335507 100.79) (end 132.7 100.79) (width 0.2) (layer B.Cu) (net 3))
   (segment (start 130.114176 102.011331) (end 131.335507 100.79) (width 0.2) (layer B.Cu) (net 3))
